File: BSE_APPS_Error_Detection/BSE_APPS_Error_Detection.brd (EAGLE design)
At the start: 100 x 63.5 mm, 21 parts, among them IC1 TLC339P, IC2 4081N, IC3 4013N

Commit message: Brandon
Brandon
Connections:
- removed net N$1: IC3.3, IC3.5
- net GND: now also IC3.3, IC3.5
Routing:
- net GND: track 207.8 -> 238.3 mm
- net N$1: track 6.47 -> 0.00 mm
Changed lines of the file:
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@@
 <?xml version="1.0" encoding="utf-8"?>
 <!DOCTYPE eagle SYSTEM "eagle.dtd">
-<eagle version="8.4.1">
+<eagle version="8.6.2">
 <drawing>
 <settings>
@@
 <wire x1="100" y1="63.49" x2="0" y2="63.49" width="0" layer="20"/>
 <wire x1="0" y1="63.49" x2="0" y2="0" width="0" layer="20"/>
+<dimension x1="0" y1="63.49" x2="0" y2="0" x3="-11.43" y3="31.745" textsize="1.778" layer="1"/>
+<dimension x1="100" y1="63.49" x2="0" y2="63.49" x3="50" y3="69.85" textsize="1.778" layer="1"/>
 </plain>
 <attributes>
@@
 <param name="checkRestrict" value="1"/>
 <param name="checkStop" value="0"/>
+<param name="checkValues" value="0"/>
 <param name="useDiameter" value="13"/>
 <param name="maxErrors" value="50"/>
@@
 <wire x1="60.96" y1="22.86" x2="63.0936" y2="20.7264" width="0.1524" layer="16"/>
 <wire x1="92.6592" y1="24.0792" x2="92.71" y2="24.13" width="0.1524" layer="16"/>
+<contactref element="IC3" pad="5"/>
+<contactref element="IC3" pad="3"/>
+<wire x1="41.91" y1="42.5196" x2="41.91" y2="41.91" width="0.1524" layer="16"/>
+<wire x1="43.5864" y1="44.196" x2="41.91" y2="42.5196" width="0.1524" layer="16"/>
+<wire x1="43.5864" y1="45.2628" x2="43.5864" y2="44.196" width="0.1524" layer="16"/>
+<wire x1="41.91" y1="46.9392" x2="43.5864" y2="45.2628" width="0.1524" layer="16"/>
+<wire x1="41.91" y1="46.9392" x2="41.91" y2="46.99" width="0.1524" layer="16"/>
+<wire x1="39.9288" y1="41.91" x2="41.91" y2="41.91" width="0.1524" layer="1"/>
+<wire x1="32.004" y1="33.9852" x2="39.9288" y2="41.91" width="0.1524" layer="1"/>
+<wire x1="22.5552" y1="33.9852" x2="32.004" y2="33.9852" width="0.1524" layer="1"/>
+<wire x1="21.59" y1="33.02" x2="22.5552" y2="33.9852" width="0.1524" layer="1"/>
 </signal>
 <signal name="BSE_HIGH">
@@
 <contactref element="SV1" pad="8"/>
 </signal>
-<signal name="N$1">
-<contactref element="IC3" pad="5"/>
-<contactref element="IC3" pad="3"/>
-<wire x1="41.91" y1="42.5196" x2="41.91" y2="41.91" width="0.1524" layer="16"/>
-<wire x1="43.5864" y1="44.196" x2="41.91" y2="42.5196" width="0.1524" layer="16"/>
-<wire x1="43.5864" y1="45.2628" x2="43.5864" y2="44.196" width="0.1524" layer="16"/>
-<wire x1="41.91" y1="46.9392" x2="43.5864" y2="45.2628" width="0.1524" layer="16"/>
-<wire x1="41.91" y1="46.9392" x2="41.91" y2="46.99" width="0.1524" layer="16"/>
-</signal>
 </signals>

Commit message: PCB Designs
Rev C
Parts:
- removed F1: FUSEBLANK_5X20MM, fuse:FUSE_HOLDER_5X20MM
- removed SV1: (no value), con-lsta:FE09W
- added F1-0.5A: FUSEBLANK_5X20MM, fuse:FUSE_HOLDER_5X20MM
- added GND: (no value), con-lsta:FE09W
- moved IN-OUT 16.6 mm to (86.4, 6.35)
- renumbered IC1 to IC1-TLC339, IC2 to IC2-CD4081, IC3 to IC3-CD4013, R1 to R1-30K, R1-APPS to R1-10K, R2 to R2-30K, R2-BSE to R2-10K, R3 to R3-30K, R4 to R4-30K, R4-APPS-BELOW to R4-10K, R5 to R5-220, R6 to R6-30K, R7 to R7-30K, R8 to R8-30K, R9 to R9-30K
Connections:
- net APPS_ACTUATED: now also GND.6; no longer SV1.6
- net APPS_HIGH: now also GND.4; no longer SV1.4
- net APPS_SIGNAL: now also GND.3; no longer SV1.3
- net BSE_HIGH: now also GND.5; no longer SV1.5
- net BSE_SIGNAL: now also GND.2; no longer SV1.2
- net ERROR: now also GND.7; no longer SV1.7
- net GND: now also GND.1; no longer SV1.1
- net LATCED: now also GND.8; no longer SV1.8
- net N$8: now also F1-0.5A.2; no longer F1.2
- net VCC: now also F1-0.5A.1, GND.9; no longer F1.1, SV1.9
Routing:
- net APPS_HIGH: track 81.3 -> 124.6 mm
- net ERROR: track 54.3 -> 92.3 mm
- net VCC: track 187.0 -> 158.2 mm, vias 0 -> 1
- net APPS_ACTUATED: track 71.5 -> 99.6 mm, vias 0 -> 3
- net GND: track 238.3 -> 214.9 mm, vias 0 -> 1
- net APPS_SIGNAL: track 72.2 -> 90.9 mm
- net N$3: track 66.1 -> 81.5 mm, vias 0 -> 1
- net N$8: track 47.0 -> 61.4 mm
- net N$11: track 80.8 -> 94.1 mm
- net VSS: track 23.2 -> 33.4 mm
- net LATCHED: track 97.2 -> 101.3 mm, vias 0 -> 2
- net BSE_SIGNAL: track 111.5 -> 115.2 mm, vias 1 -> 3
- net N$4: track 78.0 -> 79.5 mm, vias 1 -> 3
- net N$7: track 42.6 -> 43.3 mm
- net BSE_HIGH: track 104.3 -> 104.2 mm, vias 1 -> 0
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- added copper zone on layer 1, net N$1
- added copper zone on layer 16, net N$2
Other:
- board size 100 x 63.5 mm -> 100 x 59.7 mm
- board text added: "APPS"
- board text added: "APPS BEL"
- board text added: "Ac H"
- board text added: "Ac L"
- board text added: "BS H"
- board text added: "BSE"
- board text added: "ERR"
- board text added: "GND"
- board text added: "OUT"
- board text added: "SIG"
- board text added: "Sig"
- board text added: "VCC"
