File: BSE_APPS_Error_Detection/BSE_APPS_Error_Detection.brd (EAGLE design)
At the start: 100 x 59.7 mm, 22 parts, among them IC1-TLC339 TLC339P, IC2-CD4081 4081N, IC3-CD4013 4013N, IC4-4072 4072N, IC4-TLC393 TLC393P

Commit message: Brandon update.
Changed lines of the file:
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@@
 <layer number="44" name="Drills" color="7" fill="1" visible="no" active="yes"/>
 <layer number="45" name="Holes" color="7" fill="1" visible="yes" active="yes"/>
-<layer number="46" name="Milling" color="3" fill="1" visible="no" active="yes"/>
+<layer number="46" name="Milling" color="3" fill="1" visible="yes" active="yes"/>
 <layer number="47" name="Measures" color="7" fill="1" visible="yes" active="yes"/>
 <layer number="48" name="Document" color="7" fill="1" visible="yes" active="yes"/>
@@
 <hole x="2.54" y="2.54" drill="1"/>
 <hole x="96.52" y="2.54" drill="1"/>
-<hole x="97.79" y="57.15" drill="1"/>
+<hole x="96.52" y="57.15" drill="1"/>
 <text x="86.36" y="33.02" size="1.27" layer="25">BSE</text>
 <text x="86.36" y="17.78" size="1.27" layer="25">APPS</text>
@@
 <text x="33.02" y="24.13" size="1.016" layer="25">4606X-101-562LF </text>
 <text x="30.48" y="7.62" size="1.778" layer="25">0.5A</text>
+<wire x1="2.54" y1="57.15" x2="-22.86" y2="57.15" width="0.1524" layer="47"/>
+<wire x1="-22.86" y1="57.15" x2="-22.86" y2="2.54" width="0.1524" layer="47"/>
+<wire x1="-22.86" y1="2.54" x2="2.54" y2="2.54" width="0.1524" layer="47"/>
+<wire x1="2.54" y1="2.54" x2="2.54" y2="-10.16" width="0.1524" layer="47"/>
+<wire x1="2.54" y1="-10.16" x2="96.52" y2="-10.16" width="0.1524" layer="47"/>
+<wire x1="96.52" y1="-10.16" x2="96.52" y2="2.54" width="0.1524" layer="47"/>
+<dimension x1="-22.86" y1="57.15" x2="-22.86" y2="2.54" x3="-30.48" y3="29.845" textsize="1.778" layer="47"/>
+<dimension x1="2.54" y1="-10.16" x2="96.52" y2="-10.16" x3="49.53" y3="-8.89" textsize="1.778" layer="47"/>
+<dimension x1="97.79" y1="57.65" x2="97.79" y2="56.65" x3="111.76" y3="57.15" textsize="1.778" layer="47" dtype="diameter"/>
+<wire x1="97.79" y1="57.15" x2="119.38" y2="57.15" width="0.1524" layer="47"/>
+<wire x1="119.38" y1="57.15" x2="119.38" y2="2.54" width="0.1524" layer="47"/>
+<wire x1="119.38" y1="2.54" x2="96.52" y2="2.54" width="0.1524" layer="47"/>
+<dimension x1="119.38" y1="57.15" x2="119.38" y2="2.54" x3="127" y3="29.845" textsize="1.778" layer="47"/>
+<wire x1="2.54" y1="57.15" x2="2.54" y2="2.54" width="0.1524" layer="47"/>
+<wire x1="2.54" y1="2.54" x2="96.52" y2="2.54" width="0.1524" layer="47"/>
+<wire x1="96.52" y1="2.54" x2="96.52" y2="57.15" width="0.1524" layer="47"/>
+<wire x1="96.52" y1="57.15" x2="2.54" y2="57.15" width="0.1524" layer="47"/>
+<dimension x1="2.54" y1="57.15" x2="96.52" y2="57.15" x3="49.53" y3="67.31" textsize="1.778" layer="47"/>
+<dimension x1="2.54" y1="57.15" x2="2.54" y2="2.54" x3="-30.48" y3="29.845" textsize="1.778" layer="47"/>
 </plain>
 <attributes>
