File: BSE_APPS_Error_Detection/BSE_APPS_Error_Detection.sch (EAGLE design)
At the start: 21 parts, among them IC1 TLC339P, IC2 4081N, IC3 4013N

Commit message: Brandon
Brandon
Connections:
- removed net N$1: IC3A.CLK, IC3A.D
- net GND: now also IC3A.CLK, IC3A.D
Changed lines of the file:
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@@
 <?xml version="1.0" encoding="utf-8"?>
 <!DOCTYPE eagle SYSTEM "eagle.dtd">
-<eagle version="8.4.1">
+<eagle version="8.6.2">
 <drawing>
 <settings>
@@
 <label x="193.04" y="96.52" size="1.778" layer="95" rot="R270" xref="yes"/>
 </segment>
+<segment>
+<pinref part="IC3" gate="A" pin="D"/>
+<pinref part="IC3" gate="A" pin="CLK"/>
+<wire x1="114.3" y1="71.12" x2="114.3" y2="68.58" width="0.1524" layer="91"/>
+<wire x1="114.3" y1="68.58" x2="111.76" y2="68.58" width="0.1524" layer="91"/>
+<junction x="114.3" y="68.58"/>
+<wire x1="111.76" y1="68.58" x2="111.76" y2="43.18" width="0.1524" layer="91"/>
+<label x="111.76" y="43.18" size="1.778" layer="95" rot="R270" xref="yes"/>
+</segment>
 </net>
 <net name="BSE_HIGH" class="0">
@@
 </segment>
 </net>
-<net name="N$1" class="0">
-<segment>
-<pinref part="IC3" gate="A" pin="D"/>
-<pinref part="IC3" gate="A" pin="CLK"/>
-<wire x1="114.3" y1="71.12" x2="114.3" y2="68.58" width="0.1524" layer="91"/>
-<wire x1="114.3" y1="68.58" x2="111.76" y2="68.58" width="0.1524" layer="91"/>
-<junction x="114.3" y="68.58"/>
-<wire x1="111.76" y1="68.58" x2="111.76" y2="43.18" width="0.1524" layer="91"/>
-<label x="111.76" y="43.18" size="1.778" layer="95" rot="R270" xref="yes"/>
-</segment>
-</net>

Commit message: PCB Designs
Rev C
Parts:
- renumbered F1 to F1-0.5A, IC1 to IC1-TLC339, IC2 to IC2-CD4081, IC3 to IC3-CD4013, R1 to R1-30K, R1-APPS to R1-10K, R2 to R2-30K, R2-BSE to R2-10K, R3 to R3-30K, R4 to R4-30K, R4-APPS-BELOW to R4-10K, R5 to R5-220, R6 to R6-30K, R7 to R7-30K, R8 to R8-30K, R9 to R9-30K, SV1 to GND
