File: Brake System Plausability Device/BSPD.sch (EAGLE design)
At the start: 47 parts, among them IC1 TLC339P, IC2 4081N, IC3 4013N, IC4 4093N, IC5 4013N, IC6 4069N, X1 ERR_STATE_OUT

Commit message: PCB Designs
Rev C
Parts:
- removed C5: 47uF, rcl:C-US050-024X044
- removed LED1: (no value), led:LED5MM
- removed R11: 43k, rcl:R-US_0207/12
- removed R16, R28: 30k, rcl:R-US_0207/12
- removed R8: 220, rcl:R-US_0207/12
- added C5-47UF: 47uF, rcl:C-US050-024X044
- added R11-43K: 43k, rcl:R-US_0207/12
- added R16-30K, R28-30K: 30k, rcl:R-US_0207/12
- renumbered C1 to C1-330UF, C2 to C2-47UF, C4 to C4-47UF, F1 to F1-0.5A, IC1 to IC1-TLC339, IC2 to IC2-4081, IC3 to IC3-4013, IC4 to IC4-4093, IC5 to IC5-4013, IC6 to IC6-4069, R1 to R1-10K, R10 to R10-30K, R12 to R12-43K, R14 to R14-43K, R15 to R15-30K, R17 to R17-30K, R19 to R19-220, R2 to R2-10K, R20 to R20-30K, R21 to R21-220, R22 to R22-220, R23 to R23-30K, R24 to R24-30K, R25 to R25-30K, R26 to R26-30K, R27 to R27-30K, R3 to R3-1K, R4 to R4-10K, R5 to R5-30K, R6 to R6-30K, R7 to R7-30K, R9 to R9-30K, SV2 to GND, X1 to ERR_STATE_OUT
Connections:
- removed net N$16: IC2-4081B.O, R28.2, R8.2
- removed net N$17: LED1.A, R8.1
- net BMS: now also IC5-4013A.S
- net BMS_RST: now also R16-30K.2; no longer R16.2
- net ERROR_2: now also R28-30K.2; no longer IC2-4081B.I0
- net ESO_BMS_RST: now also C5-47UF.1, R11-43K.1; no longer C5.1, R11.1
- net GND: now also C5-47UF.2, R16-30K.1, R28-30K.1; no longer C5.2, LED1.C, R16.1, R28.1
- net IMD: no longer IC5-4013A.S
- net VCC: now also R11-43K.2; no longer IC2-4081B.I1, R11.2
