File: HVAL TSAL/HVAL_TSAL.brd (EAGLE design)
At the start: 101.3 x 83.8 mm, 18 parts, among them IC1 LM555N, X2 22-23-2031

Commit message: Brandon
Brandon
Parts:
- removed C4: (no value), rcl:C102-043X133
- moved SV1 55.7 mm to (57.1, 76.2), turned to 0 degrees
- moved D6 55.0 mm to (86.4, 71.1), turned to 0 degrees
- moved R5 52.5 mm to (88.9, 62.2), turned to 0 degrees
- moved C6 51.4 mm to (58.4, 68.6), turned to 0 degrees
- moved C1 51.1 mm to (74.9, 72.4), turned to 0 degrees
- moved IN 50.9 mm to (8.89, 6.35)
- moved D5 38.1 mm to (8.89, 72.4), turned to 0 degrees
- moved C2 29.6 mm to (43.2, 72.4), turned to 0 degrees
- moved C5 29.6 mm to (47.0, 15.2), turned to 180 degrees
- moved U$1 27.0 mm to (50.8, 34.3)
- moved R3 26.5 mm to (68.6, 62.2), turned to 0 degrees
- moved C3 23.6 mm to (43.2, 5.08), turned to 180 degrees
- moved R2 20.4 mm to (45.7, 62.2)
- moved X2 19.7 mm to (29.2, 74.9), turned to 180 degrees
- moved IC1 17.8 mm to (27.9, 63.5), turned to 0 degrees
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Connections:
- net LOW_SIDE_NEG: no longer C4.2
- net N$2: no longer C4.1
Routing:
- net LOW_SIDE_NEG: track 200.3 -> 126.0 mm
- net HVAL_IN: track 9.46 -> 58.8 mm
- net N$10: track 19.6 -> 53.9 mm
- net LOW_SIDE_POS: track 149.7 -> 129.1 mm
- net TSAL_OUT: track 83.4 -> 69.6 mm
- net N$3: track 25.5 -> 37.5 mm
- net N$2: track 64.5 -> 53.0 mm
- net N$1: track 59.9 -> 49.2 mm
- net TSAL_IN: track 8.66 -> 13.9 mm
Other:
- board size 101.3 x 83.8 mm -> 100 x 80 mm
- board text added: "Blinky"
- board text added: "HIGH"
- board text added: "LOW"
- board text added: "Steady"
- board text added: "VOLTAGE"
- board text removed: "HIGH VOLTAGE AREA"
- board text removed: "LOW VOLTAGE AREA"

Commit message: PCB Designs
Rev C
Parts:
- removed D5, D6: HLMP6, display-hp:HLMP6
- added LED1, LED2: (no value), led:LED3MM
- C3-22UF: value (none) -> 22uF
- C5-0.1UF: value (none) -> 0.1uF
- C6-220UF: value (none) -> 220uF
- renumbered C1 to C1-0.47UF, C2 to C2-0.15UF, C3 to C3-22UF, C5 to C5-0.1UF, C6 to C6-220UF, F1 to F1-1.6A, IC1 to IC1-LM555, R1 to R1-66K, R2 to R2-350, R3 to R3-100, R5 to R5-100
Connections:
- net HVAL_IN: now also LED2.A; no longer D5.A
- net LOW_SIDE_NEG: now also LED1.K, LED2.K; no longer D5.K, D6.K
- net TSAL_IN: now also LED1.A; no longer D6.A
Routing:
- net HVAL_IN: track 58.8 -> 86.9 mm
- net TSAL_IN: track 13.9 -> 12.6 mm
- net LOW_SIDE_NEG: track 126.0 -> 125.4 mm
- added copper zone on layer 1, net N$4
- added copper zone on layer 16, net N$5
Other:
- board text added: "GND"
- board text added: "HV+"
- board text added: "HV-"
- board text added: "HVAL"
- board text added: "TSAL"
- board text added: "VCC"
