File: HVAL TSAL/HVAL_TSAL.brd (EAGLE design)
At the start: 100 x 80 mm, 17 parts, among them IC1-LM555 LM555N, X1 22-23-2021

Commit message: Brandon update.
Parts:
- removed R3, R5: 220, resistor:0309/12
- added C4: 22uF, rcl:C150-091X182
- added C7: 0.1uF, rcl:E7,5-16
- added C8: 220uF, rcl:C050-055X075
- added F2, F3: FUSEBLANK_5X20MM, fuse:FUSE_HOLDER_5X20MM
- added IC1: 4081N, 40xx:DIL14
- added IC2: 4030N, 40xx:DIL14
- added LED3: (no value), led:LED3MM
- added RN1: 33k, resistor-sil:SIL9
- added RN2: 470, resistor-sil:SIL4
- added U$2: EPM1205SJ, DC-DC Converter:EPM1205SJ
- added X2: 22-23-2021 -Pow, con-molex:22-23-2021
- OUT: value 22-23-2031 -> 22-27-2061-06; device con-molex:22-23-2031 -> con-molex:6410-06
- VCC: device con-lsta:FE05W -> con-lsta:FE10
- X1: value 22-23-2021 -> 22-23-2021 - AIRS
- moved LED2 88.9 mm to (73.7, 11.4)
- moved OUT 86.4 mm to (94.0, 17.8), turned to 90 degrees
- moved R1 80.7 mm to (82.5, 22.9), turned to 90 degrees
- moved VCC 78.3 mm to (83.8, 2.54)
- moved C3 72.2 mm to (26.7, 73.7), turned to 0 degrees
- moved C5 71.9 mm to (25.4, 58.4), turned to 0 degrees
- moved IC1-LM555 65.6 mm to (86.4, 40.6), turned to 90 degrees
- moved C2 61.0 mm to (74.9, 20.3), turned to 90 degrees
- moved LED1 60.2 mm to (80.0, 11.4)
- moved X1 59.7 mm to (7.62, 74.9), turned to 0 degrees
- moved F1 58.9 mm to (7.62, 64.8), turned to 270 degrees
- moved C1 50.9 mm to (74.9, 52.1), turned to 90 degrees
- moved U$1 34.2 mm to (53.3, 62.2), turned to 0 degrees
- moved R2 29.5 mm to (74.9, 66.0), turned to 90 degrees
- moved C6 19.1 mm to (74.9, 41.9), turned to 90 degrees
Connections:
- net HIGH_SIDE_NEG renamed AIRS_L
- net HIGH_SIDE_POS renamed AIRS_H
- removed net LOW_SIDE_NEG: C1.2, C2.2, C6.2, IC1-LM555.1, LED1.K, LED2.K, OUT.3, U$1.7, VCC.1
- removed net LOW_SIDE_POS: C6.1, IC1-LM555.4, IC1-LM555.8, OUT.1, R1.1, R5.1, U$1.5, VCC.5
- removed net TSAL_IN: LED1.A, R5.2
- new net 0: OUT.5, VCC.2
- new net AIRS_CLSD_H: C6.1, IC1.2, IC2.1, U$1.5, VCC.6
- new net AIRS_CLSD_L: C6.2, U$1.7
- new net GND: C1.2, C2.2, C8.2, IC1-LM555.1, IC1.12, IC1.13, IC1.5, IC1.6, IC1.7, IC1.8, IC1.9, IC2.7, OUT.3, RN1.1, RN2.1, U$2.7, VCC.1
- new net GREEN: IC2.3, LED3.A, OUT.6, RN1.2, VCC.7
- new net N$11: IC2.11, RN1.7
- new net N$14: LED1.K, RN2.3
- new net N$15: LED3.K, RN2.4
- new net N$2: IC2.10, RN1.6
- new net N$3: IC1.11, RN1.5
- new net N$4: F2.1, X2.2
- new net N$5: F3.2, OUT.4
- new net N$6: IC1.10, RN1.4
- new net N$8: IC2.4, RN1.9
- new net N$9: IC1.4, RN1.8
- new net POWER_H: C4.1, C7.+, F2.2, U$2.12
- new net POWER_L: C4.2, C7.-, U$2.10, X2.1
- new net RED: IC1-LM555.4, IC1.3, LED1.A, OUT.1, R1.1, RN1.3, VCC.8
- new net VCC: C8.1, IC1-LM555.8, IC1.14, IC2.12, IC2.13, IC2.14, IC2.5, IC2.6, IC2.8, IC2.9, U$2.5, VCC.10
- new net VDD: F3.1, IC1.1, IC2.2, VCC.9
- net DIS: now also VCC.4; no longer VCC.3
- net N$1: now also LED2.K, RN2.2; no longer LED2.A, R3.1
- net TR_THR: now also VCC.3; no longer VCC.2
- net TSAL_OUT: now also LED2.A, VCC.5; no longer R3.2, VCC.4
Routing:
- net LOW_SIDE_NEG: track 187.4 -> 0.00 mm, vias 1 -> 0
- net GND: track 0.00 -> 175.6 mm, vias 0 -> 1
- net LOW_SIDE_POS: track 168.3 -> 0.00 mm
- net VCC: track 0.00 -> 133.5 mm, vias 0 -> 1
- net RED: track 0.00 -> 126.5 mm, vias 0 -> 1
- net GREEN: track 0.00 -> 100.5 mm
- net AIRS_CLSD_H: track 0.00 -> 91.5 mm
- net VDD: track 0.00 -> 78.6 mm
- net POWER_L: track 0.00 -> 65.3 mm
- net POWER_H: track 0.00 -> 58.1 mm
- net N$1: track 72.7 -> 18.0 mm
- net AIRS_L: track 97.5 -> 58.2 mm
- net AIRS_H: track 99.6 -> 60.3 mm
- net TR_THR: track 53.5 -> 92.4 mm
- net AIRS_CLSD_L: track 0.00 -> 34.5 mm
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- added copper zone on layer 1, net N$12
- added copper zone on layer 16, net N$13
- removed copper zone on layer 1, net N$2
- removed copper zone on layer 16, net N$3
Other:
- board text added: "+12V"
- board text added: "+60V in"
- board text added: "0.15uF"
- board text added: "0.1uF"
- board text added: "0.47uF"
- board text added: "1.6A"
- board text added: "220uF"
- board text added: "22uF"
- board text added: "330k"
- board text added: "33k"
- board text added: "470"
- board text added: "6.8k"
- board text added: "AIRS_H"
- board text added: "AIRS_L"
- board text added: "CD4030N"
- board text added: "CD4081N"
- board text added: "GLV"
- board text added: "Green"
- board text added: "HV in"
- board text added: "HVI"
- board text added: "LM555N"
- board text added: "Nuet"
- board text added: "Nuetral"
- board text added: "Power_H"
- board text added: "Power_L"
- board text added: "Red"
- board text added: "TR/Thr"
- board text removed: "Blinky"
- board text removed: "HV+"
- board text removed: "HV-"
- board text removed: "HVAL"
- board text removed: "LOW"
- board text removed: "Steady"
- board text removed: "TR/THR"
