File: HVAL TSAL/HVAL_TSAL.sch (EAGLE design)
At the start: 18 parts, among them IC1 LM555N, X2 22-23-2031

Commit message: Brandon
Brandon
Parts:
- removed C4: (no value), rcl:C-EU102-043X133
Connections:
- net LOW_SIDE_NEG: no longer C4.2
- net N$2: no longer C4.1
Changed lines of the file:
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@@
 </class>
 <class number="1" name="High Voltage" width="0.635" drill="0.162559375">
-<clearance class="1" value="0.205"/>
+<clearance class="1" value="0.5"/>
 </class>
 </classes>
@@
 <part name="D5" library="display-hp" library_urn="urn:adsk.eagle:library:212" deviceset="HLMP6" device="" package3d_urn="urn:adsk.eagle:package:12992/1"/>
 <part name="D6" library="display-hp" library_urn="urn:adsk.eagle:library:212" deviceset="HLMP6" device="" package3d_urn="urn:adsk.eagle:package:12992/1"/>
-<part name="C4" library="rcl" library_urn="urn:adsk.eagle:library:334" deviceset="C-EU" device="102-043X133" package3d_urn="urn:adsk.eagle:package:23647/1"/>
 <part name="C3" library="rcl" library_urn="urn:adsk.eagle:library:334" deviceset="C-EU" device="150-091X182" package3d_urn="urn:adsk.eagle:package:23659/1"/>
 <part name="C5" library="rcl" library_urn="urn:adsk.eagle:library:334" deviceset="C-US" device="075-032X103" package3d_urn="urn:adsk.eagle:package:23646/1"/>
@@
 </instance>
 <instance part="D6" gate="A" x="114.3" y="-2.54"/>
-<instance part="C4" gate="G$1" x="-2.54" y="-27.94" rot="R90"/>
 <instance part="C3" gate="G$1" x="-33.02" y="2.54"/>
 <instance part="C5" gate="G$1" x="-22.86" y="2.54"/>
@@
 <wire x1="-50.8" y1="-2.54" x2="-33.02" y2="-2.54" width="0.1524" layer="91"/>
 <pinref part="U$1" gate="G$1" pin="10-IN-"/>
-<pinref part="C4" gate="G$1" pin="1"/>
-<wire x1="-33.02" y1="-2.54" x2="-27.94" y2="-2.54" width="0.1524" layer="91"/>
-<wire x1="-27.94" y1="-2.54" x2="-22.86" y2="-2.54" width="0.1524" layer="91"/>
+<wire x1="-33.02" y1="-2.54" x2="-22.86" y2="-2.54" width="0.1524" layer="91"/>
 <wire x1="-22.86" y1="-2.54" x2="-17.78" y2="-2.54" width="0.1524" layer="91"/>
-<wire x1="-5.08" y1="-27.94" x2="-27.94" y2="-27.94" width="0.1524" layer="91"/>
-<wire x1="-27.94" y1="-27.94" x2="-27.94" y2="-2.54" width="0.1524" layer="91"/>
-<junction x="-27.94" y="-2.54"/>
 <pinref part="C3" gate="G$1" pin="2"/>
 <junction x="-33.02" y="-2.54"/>
@@
 </segment>
 </net>
-<net name="LOW_SIDE_NEG" class="1">
+<net name="LOW_SIDE_NEG" class="0">
 <segment>
 <pinref part="IC1" gate="A" pin="GND"/>
 <pinref part="U$1" gate="G$1" pin="7-OUT-"/>
-<wire x1="17.78" y1="-2.54" x2="20.32" y2="-2.54" width="0.1524" layer="91"/>
-<pinref part="C4" gate="G$1" pin="2"/>
-<wire x1="2.54" y1="-27.94" x2="20.32" y2="-27.94" width="0.1524" layer="91"/>
-<wire x1="20.32" y1="-27.94" x2="20.32" y2="-2.54" width="0.1524" layer="91"/>
-<junction x="20.32" y="-2.54"/>
-<wire x1="20.32" y1="-2.54" x2="22.86" y2="-2.54" width="0.1524" layer="91"/>
+<wire x1="17.78" y1="-2.54" x2="22.86" y2="-2.54" width="0.1524" layer="91"/>
 <pinref part="C6" gate="G$1" pin="2"/>
 <junction x="22.86" y="-2.54"/>

Commit message: PCB Designs
Rev C
Parts:
- removed D5, D6: HLMP6, display-hp:HLMP6
- added LED1, LED2: (no value), led:LED3MM
- C3-22UF: value (none) -> 22uF
- C5-0.1UF: value (none) -> 0.1uF
- C6-220UF: value (none) -> 220uF
- renumbered C1 to C1-0.47UF, C2 to C2-0.15UF, C3 to C3-22UF, C5 to C5-0.1UF, C6 to C6-220UF, F1 to F1-1.6A, IC1 to IC1-LM555, R1 to R1-66K, R2 to R2-350, R3 to R3-100, R5 to R5-100
Connections:
- net HVAL_IN: now also LED2.A; no longer D5.A
- net LOW_SIDE_NEG: now also LED1.C, LED2.C; no longer D5.K, D6.K
- net TSAL_IN: now also LED1.A; no longer D6.A
Other:
- moved on the sheet: U$1
