File: Pedal Plausibility Device/Pedal System Circuit.brd (EAGLE design)
At the start: 81 x 57.1 mm, 19 parts, among them IC1 LM358N, IC2 TLC339P, IC3 4081N

Commit message: PCB Designs
Rev C
Parts:
- removed R3: 200, resistor:RTRIM43P
- removed R4, R9: 30k, resistor:0207/12
- removed SV1: (no value), con-lsta:FE09W
- added GND: (no value), con-lsta:FE09W
- added R3-200: 200, resistor:RTRIM43P
- added R4-30K, R9-30K: 30k, resistor:0207/12
- renumbered F1 to F1-0.5A, IC2 to IC2-TLC339, IC3 to IC3-4081, R1 to R1-10K, R10 to R10-30K, R2 to R2-2K, R5 to R5-10K, R6 to R6-10K, R7 to R7-30K, R8 to R8-10K
Connections:
- net GND: now also GND.1, R3-200.3, R9-30K.1; no longer R3.3, R9.1, SV1.1
- net HIGH: now also GND.8; no longer SV1.8
- net LOW: now also GND.7, R4-30K.2; no longer R4.2, SV1.7
- net N$4: now also R9-30K.2; no longer R9.2
- net PEDAL_1: now also GND.2; no longer SV1.2
- net PEDAL_2: now also GND.3; no longer SV1.3
- net POT_ABOVE: now also GND.4, R3-200.1; no longer R3.1, SV1.4
- net POT_BELOW: now also GND.6, R3-200.2; no longer R3.2, SV1.6
- net SUB_OUT: now also GND.5; no longer SV1.5
- net VCC: now also GND.9, R4-30K.1; no longer R4.1, SV1.9
Routing:
- net N$4: track 85.5 -> 37.7 mm
- net HIGH: track 61.3 -> 104.2 mm
- net POT_BELOW: track 88.0 -> 46.0 mm
- net PEDAL_2: track 63.9 -> 98.7 mm
- net PEDAL_1: track 78.8 -> 110.4 mm
- net GND: track 163.6 -> 133.6 mm
- net LOW: track 81.0 -> 103.6 mm
- net VCC: track 141.0 -> 158.4 mm
- net POT_ABOVE: track 63.1 -> 56.2 mm, vias 1 -> 0
- net SUB_OUT: track 103.3 -> 98.1 mm
Other:
- board text added: "GND"
- board text added: "HIGH"
- board text added: "LOW"
- board text added: "PED-1"
- board text added: "PED-2"
- board text added: "POT-H"
- board text added: "POT-L"
- board text added: "SUB-O"
- board text added: "Sig"
- board text added: "VCC"
