File: Pedal Plausibility Device/Pedal System Circuit.sch (EAGLE design)
At the start: 19 parts, among them IC1 LM358N, IC2 TLC339P, IC3 4081N

Commit message: PCB Designs
Rev C
Parts:
- renumbered F1 to F1-0.5A, IC2 to IC2-TLC339, IC3 to IC3-4081, R1 to R1-10K, R10 to R10-30K, R2 to R2-2K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
