File: Shutdown_Circuit/Shutdown Circuit.brd (EAGLE design)
At the start: 100 x 80 mm, 27 parts, among them IC1 4093N, X1 22-23-2021, X3 22-23-2081

Commit message: Brandon
Brandon
Parts:
- added IC2: 4069N, 40xx:DIL14
- added R8: (no value), resistor:0207/10
- SV1: device con-lsta:FE20W -> con-lstb:MA07-1
- X3: value 22-23-2081 -> (none); device con-molex:22-23-2081 -> con-molex:22-23-2061
- moved SV1 233.8 mm to (-17.8, -199.4)
- moved X3 67.4 mm to (-19.1, -214.6)
Connections:
- removed net N$17: IC1.3, OK7.1
- new net N$15: IC2.2, OK7.1
- new net N$8: IC1.3, IC2.1, R8.2
- net APPS_BSE: now also SV1.6; no longer SV1.19
- net BMS: now also SV1.3; no longer SV1.16
- net FROM_BTNS: now also X3.4, X3.5; no longer X3.6, X3.7
- net GND: now also R8.1, X3.1; no longer X3.5
- net IMD: now also SV1.2; no longer SV1.15
- net PPD: now also SV1.5; no longer SV1.18
- net PSBD: now also SV1.4; no longer SV1.17
- net TO_AIRS_2: now also X3.2; no longer X3.4
- net TO_BTNS: now also X3.6; no longer X3.8
- net VCC: now also SV1.7; no longer SV1.20
- net VDD: now also IC2.14
- net VSS: now also IC2.7

Commit message: Brandon
Brandon
Parts:
- R1, R10, R11, R14, R2, R6, R7: value (none) -> 240
- R12, R13, R3, R5, R8, R9: value (none) -> 30k
- R4: value 2k -> 1.2k
- X1: value 22-23-2021 -> Inputs
- X2: value (none) -> ERROR_Inputs
- X3: value (none) -> SW_AIRS_I/O
- moved SV1 283.7 mm to (49.5, 76.2)
- moved X3 259.9 mm to (77.5, 26.7)
- moved R8 257.2 mm to (11.4, 71.1)
- moved IC2 239.8 mm to (58.4, 61.0), turned to 270 degrees
- moved R6 230.2 mm to (90.2, 69.8)
- moved R4 198.0 mm to (90.2, 47.0)
- moved C1 178.6 mm to (72.4, 47.0)
- moved R2 150.4 mm to (82.5, 54.6)
- moved IC1 145.9 mm to (58.4, 38.1), turned to 270 degrees
- moved OK7 115.6 mm to (19.1, 41.9)
- moved X2 103.8 mm to (94.0, 30.5), turned to 90 degrees
- moved X1 73.7 mm to (6.35, 49.5), turned to 270 degrees
- moved R1 57.1 mm to (90.2, 64.8)
- moved OK6 49.3 mm to (19.1, 52.1)
- moved R11 41.1 mm to (90.2, 59.7)
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Connections:
- net N$12: now also OK4.2
Routing:
- net GND: track 0.00 -> 178.1 mm
- net IMD: track 0.00 -> 139.2 mm
- net N$11: track 0.00 -> 119.5 mm
- net BMS: track 0.00 -> 118.0 mm
- net N$20: track 0.00 -> 114.8 mm
- net N$14: track 0.00 -> 101.8 mm
- net APPS_BSE: track 0.00 -> 99.2 mm
- net FROM_BTNS: track 0.00 -> 98.9 mm
- net BSPD: track 0.00 -> 97.1 mm
- net VCC: track 0.00 -> 93.6 mm, vias 0 -> 1
- net TO_BTNS: track 0.00 -> 88.5 mm
- net N$16: track 0.00 -> 74.2 mm
- net N$12: track 0.00 -> 71.0 mm
- net N$8: track 0.00 -> 69.1 mm, vias 0 -> 1
- net TO_AIRS_2: track 0.00 -> 62.7 mm
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Other:
- board size 100 x 80 mm -> 100 x 61 mm

Commit message: PCB Designs
Rev C
Parts:
- removed F1: FUSEBLANK_5X20MM, fuse:FUSE_HOLDER_5X20MM
- removed IC1: 4093N, 40xx:DIL14
- removed OK1, OK2, OK3, OK4, OK5, OK6, OK7: TLP222AF, optocoupler:DIP4
- added F1-0.5A: FUSEBLANK_5X20MM, fuse:FUSE_HOLDER_5X20MM
- added IC1-CD4093: 4093N, 40xx:DIL14
- added OK1-TLP222AF, OK2-TLP222AF, OK3-TLP222AF, OK4-TLP222AF, OK5-TLP222AF, OK6-TLP222AF, OK7-TLP222AF: TLP222AF, optocoupler:DIP4
- moved X3 1.27 mm to (77.5, 25.4), turned to 180 degrees
- turned X2 to 270 degrees
- renumbered C1 to C1-440UF, IC2 to IC2-CD4069, R1 to R1-240, R10 to R10-240, R11 to R11-240, R12 to R12-30K, R13 to R13-30K, R14 to R14-240, R2 to R2-240, R3 to R3-30K, R4 to R4-1.2K, R5 to R5-30K, R6 to R6-240, R7 to R7-240, R8 to R8-30K, R9 to R9-30K
Connections:
- removed net N$20: OK7.2, R6-240.2
- new net N$20-TLP222AF: OK7-TLP222AF.2, R6-240.2
- net APPS_BSE: now also OK1-TLP222AF.1; no longer OK1.1
- net BMS: now also OK4-TLP222AF.1; no longer OK4.1
- net BSPD: now also OK3-TLP222AF.1; no longer OK3.1
- net FROM_BTNS: now also OK7-TLP222AF.4; no longer OK7.4
- net IMD: now also OK5-TLP222AF.1; no longer OK5.1
- net N$1: now also OK1-TLP222AF.2; no longer OK1.2
- net N$10: now also F1-0.5A.1; no longer F1.1
- net N$11: now also OK2-TLP222AF.1; no longer OK2.1
- net N$12: now also OK4-TLP222AF.2; no longer OK4.2
- net N$14: now also OK6-TLP222AF.1; no longer OK6.1
- net N$15: now also OK7-TLP222AF.1; no longer OK7.1
- net N$16: now also OK6-TLP222AF.2; no longer OK6.2
- net N$2: now also OK5-TLP222AF.3, OK6-TLP222AF.4; no longer OK5.3, OK6.4
- net N$21: now also IC1-CD4093.2; no longer IC1.2
- net N$3: now also OK4-TLP222AF.3, OK5-TLP222AF.4; no longer OK4.3, OK5.4
- net N$4: now also OK2-TLP222AF.2; no longer OK2.2
- net N$5: now also OK3-TLP222AF.3, OK4-TLP222AF.4; no longer OK3.3, OK4.4
- net N$6: now also OK2-TLP222AF.3, OK3-TLP222AF.4; no longer OK2.3, OK3.4
- net N$7: now also OK1-TLP222AF.3, OK2-TLP222AF.4; no longer OK1.3, OK2.4
- net N$8: now also IC1-CD4093.3; no longer IC1.3
- net TO_AIRS_2: now also OK7-TLP222AF.3; no longer OK7.3
- net TO_BTNS: now also OK6-TLP222AF.3; no longer OK6.3
- net VCC: now also F1-0.5A.2, IC1-CD4093.1, OK1-TLP222AF.4; no longer F1.2, IC1.1, OK1.4
- net VDD: now also IC1-CD4093.14; no longer IC1.14
- net VSS: now also IC1-CD4093.7; no longer IC1.7
Routing:
- net N$20: track 114.8 -> 0.00 mm
- net N$20-TLP222AF: track 0.00 -> 73.2 mm
- net APPS_BSE: track 99.2 -> 160.1 mm
- net TO_AIRS_2: track 62.7 -> 109.9 mm
- net TO_BTNS: track 88.5 -> 48.7 mm
- net N$15: track 60.5 -> 21.7 mm
- net BMS: track 118.0 -> 154.9 mm
- net N$14: track 101.8 -> 77.4 mm
- net N$12: track 71.0 -> 55.7 mm, vias 0 -> 1
- net IMD: track 139.2 -> 124.4 mm, vias 0 -> 1
- net N$16: track 74.2 -> 59.9 mm, vias 0 -> 1
- net VSS: track 24.3 -> 38.4 mm
- net N$8: track 69.1 -> 82.1 mm, vias 1 -> 2
- net VCC: track 93.6 -> 106.6 mm, vias 1 -> 0
- net N$7: track 14.5 -> 24.8 mm
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- added copper zone on layer 1, net N$17
- added copper zone on layer 16, net N$18
Other:
- board text added: "APPS/BSE"
- board text added: "BMS"
- board text added: "BSPD"
- board text added: "F_TSMS"
- board text added: "GND"
- board text added: "IMD"
- board text added: "In AIR-1"
- board text added: "PCM"
- board text added: "PPD"
- board text added: "To AIR-2"
- board text added: "To_BTNS"
- board text added: "VCC"
- board text added: "to AIR-1"
