File: Shutdown_Circuit/Shutdown Circuit.sch (EAGLE design)
At the start: 27 parts, among them IC1 4093N, X1 22-23-2021, X3 22-23-2081

Commit message: Brandon
Brandon
Parts:
- added IC2: 4069N, 40xx:4069N
- added R8: (no value), resistor:R-US_0207/10
- SV1: device con-lsta:FE20W -> con-lstb:MA07-1
- X3: value 22-23-2081 -> (none); device con-molex:22-23-2081 -> con-molex:22-23-2061
Connections:
- removed net N$17: IC1A.O, OK7.A
- new net N$15: IC2A.O, OK7.A
- new net N$8: IC1A.O, IC2A.I, R8.2
- net APPS_BSE: now also SV1.6; no longer SV1.19
- net BMS: now also SV1.3; no longer SV1.16
- net FROM_BTNS: now also X3-4.S, X3-5.S; no longer X3-6.S, X3-7.S
- net GND: now also R8.1, X3-1.S; no longer X3-5.S
- net IMD: now also SV1.2; no longer SV1.15
- net PPD: now also SV1.5; no longer SV1.18
- net PSBD: now also SV1.4; no longer SV1.17
- net TO_AIRS_2: now also X3-2.S; no longer X3-4.S
- net TO_BTNS: now also X3-6.S; no longer X3-8.S
- net VCC: now also SV1.7; no longer SV1.20
Other:
- note added: "0.5A FUSE"
- note added: "IN FROM TSMS"
- note added: "INPUT FROM AIRS-1"
- note added: "INPUT FROM AIRS-2"
- note added: "TO AIRS-1"
- note added: "TO AIRS-2"
- note added: "TO EXTERNAL BTNS/SWS"
- note removed: "Input from AIRS-1"
- note removed: "Input from AIRS-2"
- moved on the sheet: X3-1, X3-2, X3-3, X3-4, X3-5, X3-6

Commit message: Brandon
Brandon
Parts:
- R1, R10, R11, R14, R2, R6, R7: value (none) -> 240
- R12, R13, R3, R5, R8, R9: value (none) -> 30k
- R4: value 2k -> 1.2k
- X1: value 22-23-2021 -> Inputs
- X2: value (none) -> ERROR_Inputs
- X3: value (none) -> SW_AIRS_I/O
Connections:
- net N$12: now also OK4.C
Changed lines of the file:
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@@
 <parts>
 <part name="F1" library="fuse" library_urn="urn:adsk.eagle:library:233" deviceset="FUSE" device="BLANK_5X20MM" package3d_urn="urn:adsk.eagle:package:14079/1"/>
-<part name="R1" library="resistor" library_urn="urn:adsk.eagle:library:348" deviceset="R-US_" device="0207/10" package3d_urn="urn:adsk.eagle:package:25939/1"/>
-<part name="R7" library="resistor" library_urn="urn:adsk.eagle:library:348" deviceset="R-US_" device="0207/10" package3d_urn="urn:adsk.eagle:package:25939/1"/>
-<part name="R9" library="resistor" library_urn="urn:adsk.eagle:library:348" deviceset="R-US_" device="0207/10" package3d_urn="urn:adsk.eagle:package:25939/1"/>
-<part name="R12" library="resistor" library_urn="urn:adsk.eagle:library:348" deviceset="R-US_" device="0207/10" package3d_urn="urn:adsk.eagle:package:25939/1"/>
-<part name="R13" library="resistor" library_urn="urn:adsk.eagle:library:348" deviceset="R-US_" device="0207/10" package3d_urn="urn:adsk.eagle:package:25939/1"/>
+<part name="R1" library="resistor" library_urn="urn:adsk.eagle:library:348" deviceset="R-US_" device="0207/10" package3d_urn="urn:adsk.eagle:package:25939/1" value="240"/>
+<part name="R7" library="resistor" library_urn="urn:adsk.eagle:library:348" deviceset="R-US_" device="0207/10" package3d_urn="urn:adsk.eagle:package:25939/1" value="240"/>
+<part name="R9" library="resistor" library_urn="urn:adsk.eagle:library:348" deviceset="R-US_" device="0207/10" package3d_urn="urn:adsk.eagle:package:25939/1" value="30k"/>
+<part name="R12" library="resistor" library_urn="urn:adsk.eagle:library:348" deviceset="R-US_" device="0207/10" package3d_urn="urn:adsk.eagle:package:25939/1" value="30k"/>
+<part name="R13" library="resistor" library_urn="urn:adsk.eagle:library:348" deviceset="R-US_" device="0207/10" package3d_urn="urn:adsk.eagle:package:25939/1" value="30k"/>
 <part name="OK1" library="optocoupler" library_urn="urn:adsk.eagle:library:320" deviceset="SFH618?*" device="A" package3d_urn="urn:adsk.eagle:package:21960/1" technology="-4" value="TLP222AF"/>
 <part name="OK2" library="optocoupler" library_urn="urn:adsk.eagle:library:320" deviceset="SFH618?*" device="A" package3d_urn="urn:adsk.eagle:package:21960/1" technology="-4" value="TLP222AF "/>
@@
 <part name="OK4" library="optocoupler" library_urn="urn:adsk.eagle:library:320" deviceset="SFH618?*" device="A" package3d_urn="urn:adsk.eagle:package:21960/1" technology="-4" value="TLP222AF "/>
 <part name="OK5" library="optocoupler" library_urn="urn:adsk.eagle:library:320" deviceset="SFH618?*" device="A" package3d_urn="urn:adsk.eagle:package:21960/1" technology="-4" value="TLP222AF "/>
-<part name="R3" library="resistor" library_urn="urn:adsk.eagle:library:348" deviceset="R-US_" device="0207/10" package3d_urn="urn:adsk.eagle:package:25939/1"/>
-<part name="R5" library="resistor" library_urn="urn:adsk.eagle:library:348" deviceset="R-US_" device="0207/10" package3d_urn="urn:adsk.eagle:package:25939/1"/>
-<part name="R10" library="resistor" library_urn="urn:adsk.eagle:library:348" deviceset="R-US_" device="0207/10" package3d_urn="urn:adsk.eagle:package:25939/1"/>
-<part name="R11" library="resistor" library_urn="urn:adsk.eagle:library:348" deviceset="R-US_" device="0207/10" package3d_urn="urn:adsk.eagle:package:25939/1"/>
-<part name="R14" library="resistor" library_urn="urn:adsk.eagle:library:348" deviceset="R-US_" device="0207/10" package3d_urn="urn:adsk.eagle:package:25939/1"/>
+<part name="R3" library="resistor" library_urn="urn:adsk.eagle:library:348" deviceset="R-US_" device="0207/10" package3d_urn="urn:adsk.eagle:package:25939/1" value="30k"/>
+<part name="R5" library="resistor" library_urn="urn:adsk.eagle:library:348" deviceset="R-US_" device="0207/10" package3d_urn="urn:adsk.eagle:package:25939/1" value="30k"/>
+<part name="R10" library="resistor" library_urn="urn:adsk.eagle:library:348" deviceset="R-US_" device="0207/10" package3d_urn="urn:adsk.eagle:package:25939/1" value="240"/>
+<part name="R11" library="resistor" library_urn="urn:adsk.eagle:library:348" deviceset="R-US_" device="0207/10" package3d_urn="urn:adsk.eagle:package:25939/1" value="240"/>
+<part name="R14" library="resistor" library_urn="urn:adsk.eagle:library:348" deviceset="R-US_" device="0207/10" package3d_urn="urn:adsk.eagle:package:25939/1" value="240"/>
 <part name="OK6" library="optocoupler" library_urn="urn:adsk.eagle:library:320" deviceset="SFH618?*" device="A" package3d_urn="urn:adsk.eagle:package:21960/1" technology="-4" value="TLP222AF "/>
-<part name="X2" library="con-molex" library_urn="urn:adsk.eagle:library:165" deviceset="22-23-2061" device=""/>
-<part name="X1" library="con-molex" library_urn="urn:adsk.eagle:library:165" deviceset="22-23-2021" device=""/>
-<part name="R2" library="resistor" library_urn="urn:adsk.eagle:library:348" deviceset="R-US_" device="0207/10" package3d_urn="urn:adsk.eagle:package:25939/1"/>
+<part name="X2" library="con-molex" library_urn="urn:adsk.eagle:library:165" deviceset="22-23-2061" device="" value="ERROR_Inputs"/>
+<part name="X1" library="con-molex" library_urn="urn:adsk.eagle:library:165" deviceset="22-23-2021" device="" value="Inputs"/>
+<part name="R2" library="resistor" library_urn="urn:adsk.eagle:library:348" deviceset="R-US_" device="0207/10" package3d_urn="urn:adsk.eagle:package:25939/1" value="240"/>
 <part name="OK7" library="optocoupler" library_urn="urn:adsk.eagle:library:320" deviceset="SFH618?*" device="A" package3d_urn="urn:adsk.eagle:package:21960/1" technology="-4" value="TLP222AF "/>
 <part name="IC1" library="40xx" library_urn="urn:adsk.eagle:library:80" deviceset="4093" device="N" package3d_urn="urn:adsk.eagle:package:820/2"/>
 <part name="C1" library="resistor" library_urn="urn:adsk.eagle:library:348" deviceset="C-US" device="050-045X075" package3d_urn="urn:adsk.eagle:package:26165/1" value="440uF"/>
-<part name="R4" library="resistor" library_urn="urn:adsk.eagle:library:348" deviceset="R-US_" device="0207/12" package3d_urn="urn:adsk.eagle:package:25938/1" value="2k"/>
-<part name="R6" library="resistor" library_urn="urn:adsk.eagle:library:348" deviceset="R-US_" device="0207/10" package3d_urn="urn:adsk.eagle:package:25939/1"/>
+<part name="R4" library="resistor" library_urn="urn:adsk.eagle:library:348" deviceset="R-US_" device="0207/12" package3d_urn="urn:adsk.eagle:package:25938/1" value="1.2k"/>
+<part name="R6" library="resistor" library_urn="urn:adsk.eagle:library:348" deviceset="R-US_" device="0207/10" package3d_urn="urn:adsk.eagle:package:25939/1" value="240"/>
 <part name="IC2" library="40xx" library_urn="urn:adsk.eagle:library:80" deviceset="4069" device="N" package3d_urn="urn:adsk.eagle:package:820/2"/>
-<part name="R8" library="resistor" library_urn="urn:adsk.eagle:library:348" deviceset="R-US_" device="0207/10" package3d_urn="urn:adsk.eagle:package:25939/1"/>
+<part name="R8" library="resistor" library_urn="urn:adsk.eagle:library:348" deviceset="R-US_" device="0207/10" package3d_urn="urn:adsk.eagle:package:25939/1" value="30k"/>
 <part name="SV1" library="con-lstb" library_urn="urn:adsk.eagle:library:162" deviceset="MA07-1" device="" package3d_urn="urn:adsk.eagle:package:8341/1"/>
-<part name="X3" library="con-molex" library_urn="urn:adsk.eagle:library:165" deviceset="22-23-2061" device=""/>
+<part name="X3" library="con-molex" library_urn="urn:adsk.eagle:library:165" deviceset="22-23-2061" device="" value="SW_AIRS_I/O"/>
 </parts>
 <sheets>
@@
 </segment>
 </net>
-<net name="N$12" class="0">
-<segment>
-<pinref part="R11" gate="G$1" pin="2"/>
-<wire x1="60.96" y1="15.24" x2="55.88" y2="15.24" width="0.1524" layer="91"/>
-</segment>
-</net>
 <net name="N$13" class="0">
 <segment>
@@
 </segment>
 </net>
+<net name="N$12" class="0">
+<segment>
+<pinref part="R11" gate="G$1" pin="2"/>
+<pinref part="OK4" gate="G$1" pin="C"/>
+<wire x1="55.88" y1="15.24" x2="60.96" y2="15.24" width="0.1524" layer="91"/>
+</segment>
+</net>

Commit message: PCB Designs
Rev C
Parts:
- renumbered C1 to C1-440UF, F1 to F1-0.5A, IC1 to IC1-CD4093, IC2 to IC2-CD4069, OK1 to OK1-TLP222AF, OK2 to OK2-TLP222AF, OK3 to OK3-TLP222AF, OK4 to OK4-TLP222AF, OK5 to OK5-TLP222AF, OK6 to OK6-TLP222AF, OK7 to OK7-TLP222AF, R1 to R1-240, R10 to R10-240, R11 to R11-240, R12 to R12-30K, R13 to R13-30K, R14 to R14-240, R2 to R2-240, R3 to R3-30K, R4 to R4-1.2K, R5 to R5-30K, R6 to R6-240, R7 to R7-240, R8 to R8-30K, R9 to R9-30K
Connections:
- net N$20 renamed N$20-TLP222AF
