File: Accumulator/Accumulator Fuse Tree Diagram/12s9p_segment.sch (EAGLE design)
At the start: 232 parts

Commit message: Accumulator schematic first pass
Parts:
- removed U$1, U$2, U$3, U$4, U$5, U$6, U$7: G881A14102T3EUG881A14102T3EU, FormulaU:G881A14102T3EUG881A14102T3EU
- added F118, F119, F120, F121, F122, F123, F124, F125, F126, F127, F128, F129, F130: (no value), special:FUSE
- added SL1: (no value), con-amp-quick:M14
Connections:
- new net N$131: F118.2, SL1.1
- new net N$132: F119.2, SL1.2
- new net N$133: F120.2, SL1.3
- new net N$134: F121.2, SL1.4
- new net N$135: F122.2, SL1.5
- new net N$136: F123.2, SL1.6
- new net N$137: F124.2, SL1.7
- new net N$138: F130.2, SL1.13
- new net N$139: F129.2, SL1.12
- new net N$140: F128.2, SL1.11
- new net N$141: F127.2, SL1.10
- new net N$142: F126.2, SL1.9
- new net N$143: F125.2, SL1.8
- net N$10: now also F118.1
- net N$102: now also F128.1
- net N$112: now also F129.1
- net N$130: now also F130.1
- net N$22: now also F120.1
- net N$32: now also F121.1
- net N$42: now also F122.1
- net N$5: now also F119.1
- net N$52: now also F123.1
- net N$62: now also F124.1
- net N$72: now also F125.1
- net N$82: now also F126.1
- net N$92: now also F127.1
Other:
- note added: "Negative Terminal"
- note added: "Positive Terminal"
- note added: "Voltage Tap Plug"
