File: BeeMS/common_daughterboard/common_daughterboard-nucleo/common_daughterboard-nucleo.sch (KiCad schematic (older format))
At the start: 27 parts, among them J1 OUT_CONN, J2 TERM, J3 IN_CONN, J4 HEAD, J5 TAIL, J6 Conn_02x10_Odd_Even, Q1 BSS138, Q2 BSS138, U1 MCP2558FD-xSN

Commit message: BeeMS Common Daughterboard V0.0.1
Parts:
- added C5: 47uF, Capacitor_SMD:C_1210_3225Metric_Pad1.42x2.65mm_HandSolder, symbol Device:C
Connections:
- net +12V: now also C5.2
- net GND: now also C5.1
- net at R2.1: now also Q2.2 (S); no longer Q2.3 (D)
- net at C1.1, Q1.2 (S): now also Q2.3 (D); no longer Q2.2 (S)
Other:
- moved on the sheet: J1, J3
Changed lines of the file:
@@
 F 3 "https://www.fairchildsemi.com/datasheets/BS/BSS138.pdf" H 1550 3500 50  0001 L CNN
 	1    1550 3500
-	-1   0    0    1
+	-1   0    0    -1
 $EndComp
 $Comp
@@
 L power:+12V #PWR06
 U 1 1 5E432AE4
-P 2300 1150
-F 0 "#PWR06" H 2300 1000 50  0001 C CNN
-F 1 "+12V" H 2150 1150 50  0000 C CNN
-F 2 "" H 2300 1150 50  0001 C CNN
-F 3 "" H 2300 1150 50  0001 C CNN
-	1    2300 1150
+P 2150 1250
+F 0 "#PWR06" H 2150 1100 50  0001 C CNN
+F 1 "+12V" H 2000 1250 50  0000 C CNN
+F 2 "" H 2150 1250 50  0001 C CNN
+F 3 "" H 2150 1250 50  0001 C CNN
+	1    2150 1250
 	1    0    0    -1
 $EndComp
@@
 L power:GND #PWR05
 U 1 1 5E434C49
-P 2000 1050
-F 0 "#PWR05" H 2000 800 50  0001 C CNN
-F 1 "GND" H 2100 1050 50  0000 C CNN
-F 2 "" H 2000 1050 50  0001 C CNN
-F 3 "" H 2000 1050 50  0001 C CNN
-	1    2000 1050
-	1    0    0    -1
-$EndComp
-Text GLabel 1550 1100 2    50   Input ~ 0
+P 1850 1150
+F 0 "#PWR05" H 1850 900 50  0001 C CNN
+F 1 "GND" H 1950 1150 50  0000 C CNN
+F 2 "" H 1850 1150 50  0001 C CNN
+F 3 "" H 1850 1150 50  0001 C CNN
+	1    1850 1150
+	1    0    0    -1
+$EndComp
+Text GLabel 1400 1200 2    50   Input ~ 0
 NBR_OUT
-Text GLabel 2700 1100 0    50   Output ~ 0
+Text GLabel 2650 1200 0    50   Output ~ 0
 NBR_IN
 Wire Wire Line
-	1500 1500 1900 1500
-Wire Wire Line
-	1500 1600 2100 1600
-Wire Wire Line
-	2700 1100 2750 1100
-Text GLabel 1900 1650 3    50   BiDi ~ 0
+	1350 1600 1750 1600
+Wire Wire Line
+	1350 1700 1950 1700
+Wire Wire Line
+	2650 1200 2700 1200
+Text GLabel 1750 1750 3    50   BiDi ~ 0
 CAN_-
 Wire Wire Line
-	1900 1650 1900 1500
-Connection ~ 1900 1500
-Wire Wire Line
-	1900 1500 2750 1500
-Text GLabel 2100 1650 3    50   BiDi ~ 0
+	1750 1750 1750 1600
+Connection ~ 1750 1600
+Wire Wire Line
+	1750 1600 2700 1600
+Text GLabel 1950 1750 3    50   BiDi ~ 0
 CAN_+
 Wire Wire Line
-	2100 1650 2100 1600
-Connection ~ 2100 1600
-Wire Wire Line
-	2100 1600 2750 1600
+	1950 1750 1950 1700
+Connection ~ 1950 1700
+Wire Wire Line
+	1950 1700 2700 1700
 $Comp
 L power:GND #PWR010
 U 1 1 5E458772
-P 3150 1800
-F 0 "#PWR010" H 3150 1550 50  0001 C CNN
-F 1 "GND" H 3300 1750 50  0000 C CNN
-F 2 "" H 3150 1800 50  0001 C CNN
-F 3 "" H 3150 1800 50  0001 C CNN
-	1    3150 1800
+P 3100 1900
+F 0 "#PWR010" H 3100 1650 50  0001 C CNN
+F 1 "GND" H 3250 1850 50  0000 C CNN
+F 2 "" H 3100 1900 50  0001 C CNN
+F 3 "" H 3100 1900 50  0001 C CNN
+	1    3100 1900
 	1    0    0    -1
 $EndComp
@@
 L power:GND #PWR02
 U 1 1 5E4593FC
-P 1100 1800
-F 0 "#PWR02" H 1100 1550 50  0001 C CNN
-F 1 "GND" H 1250 1750 50  0000 C CNN
-F 2 "" H 1100 1800 50  0001 C CNN
-F 3 "" H 1100 1800 50  0001 C CNN
-	1    1100 1800
+P 950 1900
+F 0 "#PWR02" H 950 1650 50  0001 C CNN
+F 1 "GND" H 1100 1850 50  0000 C CNN
+F 2 "" H 950 1900 50  0001 C CNN
+F 3 "" H 950 1900 50  0001 C CNN
+	1    950  1900
 	1    0    0    -1
 $EndComp
@@
 	7800 3750 7750 3750
 Connection ~ 7750 3750
-NoConn ~ 2750 1400
+NoConn ~ 2700 1500
 Wire Wire Line
 	6850 4750 6850 4800
@@
 L power:PWR_FLAG #FLG01
 U 1 1 5E8D6A7A
-P 2000 850
-F 0 "#FLG01" H 2000 925 50  0001 C CNN
-F 1 "PWR_FLAG" H 2250 900 50  0000 C CNN
-F 2 "" H 2000 850 50  0001 C CNN
-F 3 "~" H 2000 850 50  0001 C CNN
-	1    2000 850
+P 1850 950
+F 0 "#FLG01" H 1850 1025 50  0001 C CNN
+F 1 "PWR_FLAG" H 1600 1000 50  0000 C CNN
+F 2 "" H 1850 950 50  0001 C CNN
+F 3 "~" H 1850 950 50  0001 C CNN
+	1    1850 950
 	1    0    0    -1
 $EndComp
@@
 L power:PWR_FLAG #FLG02
 U 1 1 5E8D8844
-P 2300 1350
-F 0 "#FLG02" H 2300 1425 50  0001 C CNN
-F 1 "PWR_FLAG" H 2550 1400 50  0000 C CNN
-F 2 "" H 2300 1350 50  0001 C CNN
-F 3 "~" H 2300 1350 50  0001 C CNN
-	1    2300 1350
+P 2150 1450
+F 0 "#FLG02" H 2150 1525 50  0001 C CNN
+F 1 "PWR_FLAG" H 2400 1500 50  0000 C CNN
+F 2 "" H 2150 1450 50  0001 C CNN
+F 3 "~" H 2150 1450 50  0001 C CNN
+	1    2150 1450
 	-1   0    0    1
 $EndComp
@@
 L Connector:RJ45_Shielded J1
 U 1 1 5E9859F5
-P 1100 1300
-F 0 "J1" H 1157 1967 50  0000 C CNN
-F 1 "OUT_CONN" H 1157 1876 50  0000 C CNN
-F 2 "Connector_RJ:RJ45_Amphenol_RJHSE5380" V 1100 1325 50  0001 C CNN
-F 3 "~" V 1100 1325 50  0001 C CNN
-	1    1100 1300
+P 950 1400
+F 0 "J1" H 1007 2067 50  0000 C CNN
+F 1 "OUT_CONN" H 1007 1976 50  0000 C CNN
+F 2 "Connector_RJ:RJ45_Amphenol_RJHSE5380" V 950 1425 50  0001 C CNN
+F 3 "~" V 950 1425 50  0001 C CNN
+	1    950  1400
 	1    0    0    -1
 $EndComp
@@
 L Connector:RJ45_Shielded J3
 U 1 1 5E98E99D
-P 3150 1300
-F 0 "J3" H 2820 1339 50  0000 R CNN
-F 1 "IN_CONN" H 2820 1248 50  0000 R CNN
-F 2 "Connector_RJ:RJ45_Amphenol_RJHSE5380" V 3150 1325 50  0001 C CNN
-F 3 "~" V 3150 1325 50  0001 C CNN
-	1    3150 1300
+P 3100 1400
+F 0 "J3" H 2770 1439 50  0000 R CNN
+F 1 "IN_CONN" H 2770 1348 50  0000 R CNN
+F 2 "Connector_RJ:RJ45_Amphenol_RJHSE5380" V 3100 1425 50  0001 C CNN
+F 3 "~" V 3100 1425 50  0001 C CNN
+	1    3100 1400
 	-1   0    0    -1
 $EndComp
 Wire Wire Line
-	1500 1200 2300 1200
-Wire Wire Line
-	2750 1300 2300 1300
-Wire Wire Line
-	2750 1000 2000 1000
-Wire Wire Line
-	1500 900  2000 900
-Wire Wire Line
-	2000 900  2000 1000
-Connection ~ 2000 900
-Wire Wire Line
-	2000 900  2750 900
-Connection ~ 2000 1000
-Wire Wire Line
-	2000 1000 1500 1000
-Wire Wire Line
-	2000 1050 2000 1000
-Wire Wire Line
-	2300 1150 2300 1200
-Connection ~ 2300 1200
-Wire Wire Line
-	2300 1200 2750 1200
-Wire Wire Line
-	2300 1300 2300 1200
-Connection ~ 2300 1300
-Wire Wire Line
-	2300 1300 1500 1300
-Wire Wire Line
-	2000 850  2000 900
-Wire Wire Line
-	2300 1350 2300 1300
-NoConn ~ 1500 1400
-Wire Wire Line
-	1550 1100 1500 1100
+	1350 1300 2150 1300
+Wire Wire Line
+	2700 1400 2150 1400
+Wire Wire Line
+	2700 1100 1850 1100
+Wire Wire Line
+	1350 1000 1850 1000
+Wire Wire Line
+	1850 1000 1850 1100
+Connection ~ 1850 1000
+Wire Wire Line
+	1850 1000 2150 1000
+Connection ~ 1850 1100
+Wire Wire Line
+	1850 1100 1350 1100
+Wire Wire Line
+	1850 1150 1850 1100
+Wire Wire Line
+	2150 1250 2150 1300
+Connection ~ 2150 1300
+Wire Wire Line
+	2150 1300 2300 1300
+Wire Wire Line
+	2150 1400 2150 1300
+Connection ~ 2150 1400
+Wire Wire Line
+	2150 1400 1350 1400
+Wire Wire Line
+	1850 950  1850 1000
+Wire Wire Line
+	2150 1450 2150 1400
+NoConn ~ 1350 1500
+Wire Wire Line
+	1400 1200 1350 1200
 $Comp
 L Mechanical:MountingHole_Pad H1
@@
 	-1   0    0    -1
 $EndComp
+$Comp
+L Device:C C5
+U 1 1 5E40173C
+P 2300 800
+F 0 "C5" H 2415 846 50  0000 L CNN
+F 1 "47uF" H 2415 755 50  0000 L CNN
+F 2 "Capacitor_SMD:C_1210_3225Metric_Pad1.42x2.65mm_HandSolder" H 2338 650 50  0001 C CNN
+F 3 "~" H 2300 800 50  0001 C CNN
+	1    2300 800
+	1    0    0    -1
+$EndComp
+Wire Wire Line
+	2300 950  2300 1300
+Connection ~ 2300 1300
+Wire Wire Line
+	2300 1300 2700 1300
+Wire Wire Line
+	2300 650  2300 600
+Wire Wire Line
+	2300 600  2150 600
+Wire Wire Line
+	2150 600  2150 1000
+Connection ~ 2150 1000
+Wire Wire Line
+	2150 1000 2700 1000
 $EndSCHEMATC
