File: Accumulator/Accumulator Schematic/Accumulator.sch (EAGLE design)
At the start: 13 parts, among them K1 E3206S, K2 E3206S, K3 E3206S

Commit message: Files from Virtual Machine
Connections:
- net TO_AIR1 renamed FROM_BTNS
- removed net FROM_AIR1: K21.1
- removed net FROM_AIR2: K11.1
- new net 0: K11.1, K21.1
- net TO_AIR2: now also K31.1
- net TO_PRECHARGE: no longer K31.1
Other:
- note added: "1.2kΩ"
- note added: "200W"
- note added: "PRECHARGE RESISTOR"
- moved on the sheet: K1, K2
Changed lines of the file:
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@@
 <layer number="97" name="Info" color="7" fill="1" visible="yes" active="yes"/>
 <layer number="98" name="Guide" color="6" fill="1" visible="yes" active="yes"/>
+<layer number="99" name="SpiceOrder" color="7" fill="1" visible="yes" active="yes"/>
 </layers>
 <schematic xreflabel="%F%N/%S.%C%R" xrefpart="/%S.%C%R">
@@
 <part name="CHASSIS_GND" library="supply1" library_urn="urn:adsk.eagle:library:371" deviceset="GND" device=""/>
 <part name="P+1" library="supply1" library_urn="urn:adsk.eagle:library:371" deviceset="VCC" device=""/>
+<part name="X_1" library="ngspice-simulation" library_urn="urn:adsk.eagle:library:527439" deviceset="GND" device=""/>
+<part name="X_2" library="ngspice-simulation" library_urn="urn:adsk.eagle:library:527439" deviceset="GND" device=""/>
 </parts>
 <sheets>
@@
 <wire x1="60.96" y1="-15.24" x2="25.4" y2="-15.24" width="0.1524" layer="95"/>
 <wire x1="25.4" y1="-15.24" x2="25.4" y2="-7.62" width="0.1524" layer="95"/>
+<text x="91.44" y="83.82" size="1.778" layer="95">PRECHARGE RESISTOR</text>
+<text x="91.44" y="81.28" size="1.778" layer="95">1.2kΩ</text>
+<text x="91.44" y="78.74" size="1.778" layer="95">200W</text>
 </plain>
 <instances>
@@
 <attribute name="VALUE" x="76.2" y="49.53" size="1.778" layer="96"/>
 </instance>
-<instance part="K1" gate="1" x="76.2" y="106.68" smashed="yes">
-<attribute name="PART" x="77.47" y="111.76" size="1.778" layer="95"/>
-</instance>
-<instance part="K1" gate="2" x="86.36" y="104.14" smashed="yes">
-<attribute name="PART" x="88.9" y="104.14" size="1.778" layer="95"/>
-</instance>
-<instance part="K2" gate="1" x="63.5" y="83.82" smashed="yes">
-<attribute name="PART" x="64.77" y="88.9" size="1.778" layer="95"/>
-</instance>
-<instance part="K2" gate="2" x="73.66" y="81.28" smashed="yes">
-<attribute name="PART" x="76.2" y="81.28" size="1.778" layer="95"/>
+<instance part="K1" gate="1" x="78.74" y="106.68" smashed="yes">
+<attribute name="PART" x="80.01" y="111.76" size="1.778" layer="95"/>
+</instance>
+<instance part="K1" gate="2" x="88.9" y="104.14" smashed="yes">
+<attribute name="PART" x="91.44" y="104.14" size="1.778" layer="95"/>
+</instance>
+<instance part="K2" gate="1" x="68.58" y="83.82" smashed="yes">
+<attribute name="PART" x="69.85" y="88.9" size="1.778" layer="95"/>
+</instance>
+<instance part="K2" gate="2" x="78.74" y="81.28" smashed="yes">
+<attribute name="PART" x="81.28" y="81.28" size="1.778" layer="95"/>
 </instance>
 <instance part="K3" gate="1" x="0" y="91.44" smashed="yes">
@@
 <attribute name="PART" x="12.7" y="88.9" size="1.778" layer="95"/>
 </instance>
-<instance part="R1" gate="G$1" x="86.36" y="81.28" smashed="yes" rot="R90"/>
+<instance part="R1" gate="G$1" x="88.9" y="81.28" smashed="yes" rot="R90"/>
 <instance part="JP1" gate="A" x="22.86" y="63.5" smashed="yes">
 <attribute name="NAME" x="21.59" y="63.5" size="1.778" layer="95" rot="R90"/>
@@
 <attribute name="VALUE" x="25.4" y="5.08" size="1.778" layer="96" rot="R180"/>
 </instance>
+<instance part="X_1" gate="G$1" x="71.12" y="116.84" smashed="yes"/>
+<instance part="X_2" gate="G$1" x="63.5" y="91.44" smashed="yes"/>
 </instances>
 <busses>
@@
 </segment>
 </net>
-<net name="LINE-" class="0">
-<segment>
-<pinref part="F1" gate="G$1" pin="2"/>
-<wire x1="86.36" y1="53.34" x2="86.36" y2="15.24" width="0.1524" layer="91"/>
-<wire x1="86.36" y1="15.24" x2="55.88" y2="15.24" width="0.1524" layer="91"/>
-<label x="58.42" y="15.24" size="1.778" layer="95" rot="R90" xref="yes"/>
-<wire x1="86.36" y1="76.2" x2="86.36" y2="71.12" width="0.1524" layer="91"/>
-<junction x="86.36" y="53.34"/>
-<pinref part="K2" gate="2" pin="P"/>
-<wire x1="86.36" y1="71.12" x2="86.36" y2="53.34" width="0.1524" layer="91"/>
-<wire x1="73.66" y1="78.74" x2="73.66" y2="71.12" width="0.1524" layer="91"/>
-<wire x1="73.66" y1="71.12" x2="86.36" y2="71.12" width="0.1524" layer="91"/>
-<junction x="86.36" y="71.12"/>
-</segment>
-</net>
 <net name="N$14" class="0">
 <segment>
@@
 <net name="TO_PRECHARGE" class="0">
 <segment>
-<pinref part="K3" gate="1" pin="1"/>
-<wire x1="0" y1="96.52" x2="0" y2="99.06" width="0.1524" layer="91"/>
-<label x="0" y="99.06" size="1.778" layer="95" rot="R90" xref="yes"/>
-</segment>
-<segment>
 <pinref part="K2" gate="1" pin="2"/>
-<wire x1="63.5" y1="76.2" x2="63.5" y2="78.74" width="0.1524" layer="91"/>
+<wire x1="68.58" y1="76.2" x2="68.58" y2="78.74" width="0.1524" layer="91"/>
+<label x="68.58" y="76.2" size="1.778" layer="95" rot="R180" xref="yes"/>
 </segment>
 </net>
 <net name="TO_AIR1" class="0">
-<segment>
-<pinref part="K3" gate="1" pin="2"/>
-<wire x1="0" y1="86.36" x2="0" y2="83.82" width="0.1524" layer="91"/>
-<label x="0" y="83.82" size="1.778" layer="95" rot="R270" xref="yes"/>
-</segment>
 <segment>
 <wire x1="27.94" y1="-15.24" x2="27.94" y2="-17.78" width="0.1524" layer="91"/>
@@
 <segment>
 <pinref part="K3" gate="2" pin="S"/>
-<wire x1="5.08" y1="93.98" x2="5.08" y2="119.38" width="0.1524" layer="91"/>
-<label x="5.08" y="119.38" size="1.778" layer="95" rot="R90" xref="yes"/>
+<wire x1="5.08" y1="93.98" x2="5.08" y2="104.14" width="0.1524" layer="91"/>
+<label x="5.08" y="104.14" size="1.778" layer="95" xref="yes"/>
 </segment>
 </net>
@@
 <segment>
 <pinref part="K1" gate="2" pin="S"/>
-<wire x1="81.28" y1="109.22" x2="81.28" y2="124.46" width="0.1524" layer="91"/>
-<label x="81.28" y="124.46" size="1.778" layer="95" rot="R180" xref="yes"/>
+<wire x1="83.82" y1="109.22" x2="83.82" y2="124.46" width="0.1524" layer="91"/>
+<label x="83.82" y="124.46" size="1.778" layer="95" rot="R180" xref="yes"/>
 </segment>
 </net>
 <net name="FROM_AIR1" class="0">
-<segment>
-<pinref part="K2" gate="1" pin="1"/>
-<wire x1="63.5" y1="88.9" x2="63.5" y2="91.44" width="0.1524" layer="91"/>
-</segment>
 <segment>
 <wire x1="33.02" y1="-15.24" x2="33.02" y2="-17.78" width="0.1524" layer="91"/>
@@
 <net name="TO_AIR2" class="0">
 <segment>
-<pinref part="K1" gate="1" pin="2"/>
-<wire x1="76.2" y1="101.6" x2="76.2" y2="99.06" width="0.1524" layer="91"/>
-<label x="76.2" y="99.06" size="1.778" layer="95" rot="R180" xref="yes"/>
-</segment>
-<segment>
 <wire x1="38.1" y1="-15.24" x2="38.1" y2="-17.78" width="0.1524" layer="91"/>
 <label x="38.1" y="-17.78" size="2.54" layer="95" rot="R270" xref="yes"/>
 </segment>
+<segment>
+<pinref part="K3" gate="1" pin="1"/>
+<wire x1="0" y1="96.52" x2="0" y2="109.22" width="0.1524" layer="91"/>
+<wire x1="0" y1="109.22" x2="71.12" y2="109.22" width="0.1524" layer="91"/>
+<wire x1="71.12" y1="109.22" x2="71.12" y2="99.06" width="0.1524" layer="91"/>
+<pinref part="K1" gate="1" pin="2"/>
+<wire x1="78.74" y1="101.6" x2="78.74" y2="99.06" width="0.1524" layer="91"/>
+<wire x1="71.12" y1="99.06" x2="78.74" y2="99.06" width="0.1524" layer="91"/>
+</segment>
 </net>
 <net name="FROM_AIR2" class="0">
-<segment>
-<pinref part="K1" gate="1" pin="1"/>
-<wire x1="76.2" y1="111.76" x2="76.2" y2="114.3" width="0.1524" layer="91"/>
-<label x="76.2" y="114.3" size="1.778" layer="95" rot="R180" xref="yes"/>
-</segment>
 <segment>
 <wire x1="43.18" y1="-15.24" x2="43.18" y2="-17.78" width="0.1524" layer="91"/>
@@
 <segment>
 <pinref part="K1" gate="2" pin="P"/>
-<wire x1="86.36" y1="86.36" x2="86.36" y2="91.44" width="0.1524" layer="91"/>
+<wire x1="88.9" y1="86.36" x2="88.9" y2="91.44" width="0.1524" layer="91"/>
 <pinref part="K2" gate="2" pin="S"/>
-<wire x1="86.36" y1="91.44" x2="86.36" y2="101.6" width="0.1524" layer="91"/>
-<wire x1="68.58" y1="86.36" x2="68.58" y2="91.44" width="0.1524" layer="91"/>
-<wire x1="68.58" y1="91.44" x2="86.36" y2="91.44" width="0.1524" layer="91"/>
-<junction x="86.36" y="91.44"/>
-</segment>
-</net>
+<wire x1="88.9" y1="91.44" x2="88.9" y2="101.6" width="0.1524" layer="91"/>
+<wire x1="73.66" y1="86.36" x2="73.66" y2="91.44" width="0.1524" layer="91"/>
+<wire x1="73.66" y1="91.44" x2="88.9" y2="91.44" width="0.1524" layer="91"/>
+<junction x="88.9" y="91.44"/>
+</segment>
+</net>
+<net name="FROM_BTNS" class="0">
+<segment>
+<pinref part="K3" gate="1" pin="2"/>
+<wire x1="0" y1="86.36" x2="0" y2="83.82" width="0.1524" layer="91"/>
+<label x="0" y="83.82" size="1.778" layer="95" rot="R270" xref="yes"/>
+</segment>
+</net>
+<net name="LINE-" class="0">
+<segment>
+<pinref part="K2" gate="2" pin="P"/>
+<wire x1="78.74" y1="78.74" x2="78.74" y2="73.66" width="0.1524" layer="91"/>
+<pinref part="F1" gate="G$1" pin="2"/>
+<wire x1="86.36" y1="53.34" x2="88.9" y2="53.34" width="0.1524" layer="91"/>
+<wire x1="88.9" y1="53.34" x2="88.9" y2="15.24" width="0.1524" layer="91"/>
+<wire x1="88.9" y1="15.24" x2="55.88" y2="15.24" width="0.1524" layer="91"/>
+<wire x1="88.9" y1="53.34" x2="88.9" y2="73.66" width="0.1524" layer="91"/>
+<junction x="88.9" y="53.34"/>
+<wire x1="88.9" y1="73.66" x2="88.9" y2="76.2" width="0.1524" layer="91"/>
+<wire x1="78.74" y1="73.66" x2="88.9" y2="73.66" width="0.1524" layer="91"/>
+<junction x="88.9" y="73.66"/>
+<label x="58.42" y="15.24" size="1.778" layer="95" rot="R90" xref="yes"/>
+</segment>
+</net>
+<net name="0" class="0">
+<segment>
+<pinref part="K1" gate="1" pin="1"/>
+<wire x1="78.74" y1="111.76" x2="78.74" y2="119.38" width="0.1524" layer="91"/>
+<pinref part="X_1" gate="G$1" pin="0"/>
+<wire x1="78.74" y1="119.38" x2="71.12" y2="119.38" width="0.1524" layer="91"/>
+<wire x1="71.12" y1="119.38" x2="71.12" y2="116.84" width="0.1524" layer="91"/>
+</segment>
+<segment>
+<pinref part="K2" gate="1" pin="1"/>
+<wire x1="68.58" y1="88.9" x2="68.58" y2="93.98" width="0.1524" layer="91"/>
+<wire x1="68.58" y1="93.98" x2="63.5" y2="93.98" width="0.1524" layer="91"/>
+<pinref part="X_2" gate="G$1" pin="0"/>
+<wire x1="63.5" y1="93.98" x2="63.5" y2="91.44" width="0.1524" layer="91"/>
+</segment>
+</net>
